Commit message: Model WIP

File: src/k9_description/urdf/k9_urdf.xacro (robot description, xacro)
@@ -74,5 +74,5 @@
       </geometry>
     </collision>
-    <xacro:box_inertia m="40.0" x="${base_length*.8}" y="${base_width}" z="${base_height/2}" o_xyz="0 0 ${base_clearance+(base_height/4)}" o_rpy="0 0 0"/>
+    <xacro:box_inertia m="27.0" x="${base_length*.8}" y="${base_width}" z="${base_height/2}" o_xyz="0 0 ${base_clearance+(base_height/4)}" o_rpy="0 0 0"/>
   </link>
   <!-- MESH -->

File: src/k9_robot/src/description/k9.urdf (robot description, URDF)
Before this commit: robot k9_robot, 11 links, 10 joints
Links:
- link base_link: mass 27.0 -> 25.0; geometry collision box size=0.43 0.18 0.295; collision box size=0.89 0.49 0.49
- link drivewhl_l_link: mass 0.3 -> 1.0
- link drivewhl_r_link: mass 0.3 -> 1.0

File: src/k9_robot/src/description/k9.urdf.xacro (robot description, xacro)
@@ -4,5 +4,5 @@
   <material name="K9_grey">
     <!-- NOTE: the model is largely transparent in RViz -->
-    <color rgba="0.25 0.25 0.25 0.3" />
+    <color rgba="0.25 0.25 0.25 1.0" />
   </material>
   <material name="perspex_red">
@@ -78,7 +78,7 @@
     <!-- Collision layout avoids wheels and mirrors head/body -->
     <collision>
-      <origin xyz="-0.119 0.0 0.315" rpy="0.0 0.0 0.0"/>
-      <geometry>
-        <box size="0.89 0.49 0.35"/>
+      <origin xyz="-0.119 0.0 0.285" rpy="0.0 0.0 0.0"/>
+      <geometry>
+        <box size="0.89 0.49 0.49"/>
       </geometry>
     </collision>
@@ -92,5 +92,5 @@
       <!-- Shift COM slightly behind wheel contact line to prevent nose tipping -->
       <origin xyz="-0.02 0 0.15" rpy="0 0 0"/>
-      <mass value="27.0"/>
+      <mass value="25.0"/>
       <inertia
         ixx="0.98230"  ixy="0.0"  ixz="0.0"
@@ -120,5 +120,5 @@
         </geometry>
       </collision>
-      <xacro:cylinder_inertia m="0.30" r="${wheel_radius}" h="${wheel_width}"/>
+      <xacro:cylinder_inertia m="1.0" r="${wheel_radius}" h="${wheel_width}"/>
     </link>
     <joint name="${prefix}_joint" type="continuous">
