Commit message: Tweaks to model

File: src/k9_robot/src/description/k9.urdf.xacro (robot description, xacro)
@@ -4,5 +4,5 @@
   <material name="K9_grey">
     <!-- NOTE: the model is largely transparent in RViz -->
-    <color rgba="0.25 0.25 0.25 0.1" />
+    <color rgba="0.25 0.25 0.25 0.3" />
   </material>
   <material name="perspex_red">
@@ -72,5 +72,5 @@
       <origin xyz="-0.5 1.905 0" rpy="0 0 ${pi}"/>
       <geometry>
-        <mesh filename="package://k9_robot/description/k9.stl" scale="0.01 0.01 0.01"/>
+        <mesh filename="file:///home/hopkira/Documents/GitHub/k9-gazebo/src/k9_description/urdf/k9.stl" scale="0.01 0.01 0.01"/>
       </geometry>
       <material name="K9_grey"/>
@@ -89,13 +89,13 @@
       </geometry>
     </collision>
-  <inertial>
-    <!-- COM aligned with wheel contact midpoint (x=0) -->
-    <origin xyz="0 0 0.33197" rpy="0 0 0"/>
-    <mass value="27.0"/>
-    <inertia
-      ixx="0.98230"  ixy="0.0"      ixz="-0.29015"
-      iyy="2.21069"  iyz="0.0"
-      izz="2.03021"/>
-  </inertial>
+    <inertial>
+      <!-- Shift COM slightly behind wheel contact line to prevent nose tipping -->
+      <origin xyz="-0.02 0 0.15" rpy="0 0 0"/>
+      <mass value="27.0"/>
+      <inertia
+        ixx="0.98230"  ixy="0.0"  ixz="0.0"
+        iyy="2.4"  iyz="0.0"
+        izz="2.03021"/>
+    </inertial>
   </link>
   <joint name="base_joint" type="fixed">
@@ -123,9 +123,9 @@
     </link>
     <joint name="${prefix}_joint" type="continuous">
-      <parent link="base_link"/>
+      <parent link="base_footprint"/>
       <child link="${prefix}_link"/>
-      <origin xyz="${x} ${y} 0.0" rpy="0 0 0"/>
+      <!-- wheel center is wheel_radius above ground -->
+      <origin xyz="${x} ${y} ${wheel_radius}" rpy="0 0 0"/>
       <axis xyz="0 1 0"/>
-      <!-- Small damping reduces wheel jitter in contact dynamics -->
       <dynamics damping="0.05" friction="0.0"/>
     </joint>

Commit message: Detailed mass analysis

File: src/k9_robot/src/description/k9.urdf.xacro (robot description, xacro)
@@ -3,5 +3,4 @@
   <!-- ===================== Materials ===================== -->
   <material name="K9_grey">
-    <!-- NOTE: the model is largely transparent in RViz -->
     <color rgba="0.25 0.25 0.25 1.0" />
   </material>
@@ -48,7 +47,9 @@
     </inertial>
   </xacro:macro>
-  <xacro:macro name="cylinder_inertia" params="m r h">
-    <inertial>
-      <origin xyz="0 0 0" rpy="0 0 0"/>
+  <!-- Cylinder inertia about its own center.
+      rpy must match the cylinder geometry orientation -->
+  <xacro:macro name="cylinder_inertia" params="m r h rpy:='0 0 0'">
+    <inertial>
+      <origin xyz="0 0 0" rpy="${rpy}"/>
       <mass value="${m}"/>
       <inertia
@@ -90,11 +91,12 @@
     </collision>
     <inertial>
-      <!-- Shift COM slightly behind wheel contact line to prevent nose tipping -->
-      <origin xyz="-0.02 0 0.15" rpy="0 0 0"/>
+      <!-- Recomputed from 5 internal mass boxes (total 25.0 kg).
+          Origin is COM expressed in base_link frame. -->
+      <origin xyz="-0.090992 0 0.177274" rpy="0 0 0"/>
       <mass value="25.0"/>
       <inertia
-        ixx="0.98230"  ixy="0.0"  ixz="0.0"
-        iyy="2.4"  iyz="0.0"
-        izz="2.03021"/>
+        ixx="1.175508"  ixy="0.0"      ixz="-0.512311"
+        iyy="2.263333"  iyz="0.0"
+        izz="1.639449"/>
     </inertial>
   </link>
@@ -120,5 +122,9 @@
         </geometry>
       </collision>
-      <xacro:cylinder_inertia m="1.0" r="${wheel_radius}" h="${wheel_width}"/>
+      <xacro:cylinder_inertia
+        m="1.0"
+        r="${wheel_radius}"
+        h="${wheel_width}"
+        rpy="${pi/2} 0 0"/>
     </link>
     <joint name="${prefix}_joint" type="continuous">
@@ -151,7 +157,9 @@
   </link>
   <joint name="caster_swivel_joint" type="continuous">
-    <parent link="base_link"/>
+    <parent link="base_footprint"/>
     <child link="caster_swivel_link"/>
-    <origin xyz="${caster_mount_x} ${caster_mount_y} ${caster_mount_z}" rpy="0 0 0"/>
+    <!-- caster_mount_z is already defined relative to axle height;
+        convert to base_footprint by adding wheel_radius -->
+    <origin xyz="${caster_mount_x} ${caster_mount_y} ${caster_mount_z + wheel_radius}" rpy="0 0 0"/>
     <axis xyz="0 0 1"/>
     <dynamics damping="0.8" friction="0.0"/>
@@ -171,5 +179,9 @@
       </geometry>
     </collision>
-    <xacro:cylinder_inertia m="0.10" r="${caster_wheel_radius}" h="${caster_wheel_width}"/>
+    <xacro:cylinder_inertia
+      m="0.10"
+      r="${caster_wheel_radius}"
+      h="${caster_wheel_width}"
+      rpy="${pi/2} 0 0"/>
   </link>
   <joint name="caster_wheel_joint" type="continuous">

Commit message: Include Pi

File: src/k9_robot/src/description/k9.urdf.xacro (robot description, xacro)
@@ -14,4 +14,5 @@
     <color rgba="1.0 1.0 1.0 1.0"/>
   </material>
+  <xacro:property name="pi" value="3.141592653589793"/>
   <!-- ===================== Robot constants ===================== -->
   <!-- Chassis dims (m) -->

Commit message: Update k9.urdf.xacro

File: src/k9_robot/src/description/k9.urdf.xacro (robot description, xacro)
@@ -5,34 +5,13 @@
   <!-- ===================================================== -->
   <material name="K9_grey">
-<<<<<<< HEAD
-    <color rgba="0.25 0.25 0.25 1.0" />
-  </material>
-  <material name="perspex_red">
-    <color rgba="1.0 0.1 0.1 1.0" />
-=======
     <color rgba="0.25 0.25 0.25 1.0"/>
->>>>>>> b2d86b1 (Fixing URDF)
   </material>
   <material name="wheel_grey">
     <color rgba="0.7 0.7 0.7 1.0"/>
   </material>
-<<<<<<< HEAD
-  <material name="white">
-    <color rgba="1.0 1.0 1.0 1.0"/>
-  </material>
-  <xacro:property name="pi" value="3.141592653589793"/>
-  <!-- ===================== Robot constants ===================== -->
-  <!-- Chassis dims (m) -->
-  <xacro:property name="base_width"  value="0.49"/>
-  <xacro:property name="base_length" value="0.81"/>
-  <xacro:property name="base_height" value="0.52"/>
-  <!-- Drive wheels (m) -->
-  <xacro:property name="wheel_radius" value="0.06939"/>
-=======
   <!-- ===================================================== -->
   <!-- Constants                                             -->
   <!-- ===================================================== -->
   <xacro:property name="wheel_radius" value="0.0694"/>
->>>>>>> b2d86b1 (Fixing URDF)
   <xacro:property name="wheel_width"  value="0.025"/>
   <xacro:property name="track"         value="0.2022"/>
@@ -53,31 +32,7 @@
     </inertial>
   </xacro:macro>
-<<<<<<< HEAD
-  <!-- Cylinder inertia about its own center.
-      rpy must match the cylinder geometry orientation -->
-  <xacro:macro name="cylinder_inertia" params="m r h rpy:='0 0 0'">
-    <inertial>
-      <origin xyz="0 0 0" rpy="${rpy}"/>
-      <mass value="${m}"/>
-      <inertia
-        ixx="${(m/12) * (3*r*r + h*h)}" ixy="0" ixz="0"
-        iyy="${(m/12) * (3*r*r + h*h)}" iyz="0"
-        izz="${(m/2) * (r*r)}"/>
-    </inertial>
-  </xacro:macro>
-  <!-- Simple “tiny inertial” for fixed-mounted accessories to keep Gazebo happy -->
-  <xacro:macro name="tiny_inertial" params="m i">
-    <inertial>
-      <origin xyz="0 0 0" rpy="0 0 0"/>
-      <mass value="${m}"/>
-      <inertia ixx="${i}" ixy="0" ixz="0" iyy="${i}" iyz="0" izz="${i}"/>
-    </inertial>
-  </xacro:macro>
-  <!-- ===================== Base frames ===================== -->
-=======
   <!-- ===================================================== -->
   <!-- Frames                                                -->
   <!-- ===================================================== -->
->>>>>>> b2d86b1 (Fixing URDF)
   <link name="base_footprint"/>
   <!-- ===================================================== -->
@@ -104,14 +59,4 @@
     <!-- CHANGED: lower + slightly rear-shift COM, and increase pitch inertia (iyy) -->
     <inertial>
-<<<<<<< HEAD
-      <!-- Recomputed from 5 internal mass boxes (total 25.0 kg).
-          Origin is COM expressed in base_link frame. -->
-      <origin xyz="-0.090992 0 0.177274" rpy="0 0 0"/>
-      <mass value="25.0"/>
-      <inertia
-        ixx="1.175508"  ixy="0.0"      ixz="-0.512311"
-        iyy="2.263333"  iyz="0.0"
-        izz="1.639449"/>
-=======
       <!-- was: -0.02 0 0.20 -->
       <origin xyz="-0.06 0 0.16"/>
@@ -123,5 +68,4 @@
         iyz="0"
         izz="1.70"/>
->>>>>>> b2d86b1 (Fixing URDF)
     </inertial>
   </link>
@@ -190,11 +134,4 @@
         </surface>
       </collision>
-<<<<<<< HEAD
-      <xacro:cylinder_inertia
-        m="1.0"
-        r="${wheel_radius}"
-        h="${wheel_width}"
-        rpy="${pi/2} 0 0"/>
-=======
       <inertial>
         <mass value="1.0"/>
@@ -204,5 +141,4 @@
           izz="0.004"/>
       </inertial>
->>>>>>> b2d86b1 (Fixing URDF)
     </link>
     <joint name="${name}_joint" type="continuous">
@@ -242,47 +178,4 @@
     <xacro:tiny_inertial m="0.5"/>
   </link>
-<<<<<<< HEAD
-  <joint name="caster_swivel_joint" type="continuous">
-    <parent link="base_footprint"/>
-    <child link="caster_swivel_link"/>
-    <!-- caster_mount_z is already defined relative to axle height;
-        convert to base_footprint by adding wheel_radius -->
-    <origin xyz="${caster_mount_x} ${caster_mount_y} ${caster_mount_z + wheel_radius}" rpy="0 0 0"/>
-    <axis xyz="0 0 1"/>
-    <dynamics damping="0.8" friction="0.0"/>
-  </joint>
-  <link name="caster_wheel_link">
-    <visual>
-      <origin xyz="0 0 0" rpy="${pi/2} 0 0"/>
-      <geometry>
-        <cylinder radius="${caster_wheel_radius}" length="${caster_wheel_width}"/>
-      </geometry>
-      <material name="wheel_grey"/>
-    </visual>
-    <collision>
-      <origin xyz="0 0 0" rpy="${pi/2} 0 0"/>
-      <geometry>
-        <cylinder radius="${caster_wheel_radius}" length="${caster_wheel_width}"/>
-      </geometry>
-    </collision>
-    <xacro:cylinder_inertia
-      m="0.10"
-      r="${caster_wheel_radius}"
-      h="${caster_wheel_width}"
-      rpy="${pi/2} 0 0"/>
-  </link>
-  <joint name="caster_wheel_joint" type="continuous">
-    <parent link="caster_swivel_link"/>
-    <child link="caster_wheel_link"/>
-    <origin xyz="${-caster_fork_offset} 0 0" rpy="0 0 0"/>
-    <axis xyz="0 1 0"/>
-    <dynamics damping="0.10" friction="0.0"/>
-  </joint>
-  <!-- ===================== Sensors / accessories (with inertials) ===================== -->
-  <link name="lidar_link">
-    <xacro:tiny_inertial m="0.05" i="1e-5"/>
-  </link>
-  <joint name="lidar_joint" type="fixed">
-=======
   <joint name="ball_caster_joint" type="fixed">
     <parent link="base_link"/>
@@ -296,5 +189,4 @@
   <link name="base_laser"><xacro:tiny_inertial m="0.05"/></link>
   <joint name="base_laser_joint" type="fixed">
->>>>>>> b2d86b1 (Fixing URDF)
     <parent link="base_link"/>
     <child link="base_laser"/>
@@ -350,6 +242,6 @@
       <max_angular_velocity>0.63</max_angular_velocity>
       <!-- CHANGED: lower accel also caps braking decel (less "nose dive") -->
-      <max_linear_acceleration>0.4</max_linear_acceleration>
-      <max_angular_acceleration>0.4</max_angular_acceleration>
+      <max_linear_acceleration>0.28</max_linear_acceleration>
+      <max_angular_acceleration>0.21</max_angular_acceleration>
       <topic>/cmd_vel</topic>
       <odom_topic>/odom</odom_topic>

Commit message: Added ears

File: src/k9_robot/src/description/k9.urdf.xacro (robot description, xacro)
@@ -9,4 +9,10 @@
   <material name="wheel_grey">
     <color rgba="0.7 0.7 0.7 1.0"/>
+  </material>
+  <material name="k9_ear_emissive">
+  <color rgba="0 0 0 1"/>
+  </material>
+  <material name="k9_beam_material">
+    <color rgba="0 1 0 1"/>
   </material>
   <!-- ===================================================== -->
@@ -197,5 +203,5 @@
       <update_rate>10</update_rate>
       <always_on>true</always_on>
-      <topic>/world/empty/model/k9_robot/ld06/scan</topic>
+      <topic>/scan</topic>
       <pose>0 0 0 0 0 0</pose>
       <visualize>true</visualize>
@@ -213,6 +219,4 @@
         </range>
       </lidar>
-      <always_on>true</always_on>
-      <visualize>true</visualize>
     </sensor>
   </gazebo>
@@ -229,4 +233,88 @@
     <origin xyz="0.206 0 0.255"/>
   </joint>
+  <!-- ******************** LEFT EAR ****************************** -->
+<link name="l_ear_link">
+  <!-- Visual (for Gazebo visualisation) -->
+  <visual name="l_ear_visual">
+    <origin xyz="0 0 0" rpy="0 0 0"/>
+    <geometry>
+      <box size="0.015 0.02 0.03"/>
+    </geometry>
+    <material name="k9_ear_emissive">
+      <ambient>0 0 0 1</ambient>
+      <diffuse>0 0 0 1</diffuse>
+      <emissive>0 0 0 1</emissive> <!-- will be driven by Gazebo -->
+    </material>
+  </visual>
+  <visual name="l_ear_beam_visual">
+    <origin xyz="1.0 0 0" rpy="0 0 0"/>
+    <geometry>
+      <cone radius="0.01" length="2.0"/>
+    </geometry>
+    <material name="k9_beam_material">
+      <ambient>0 0 0 1</ambient>
+      <diffuse>0 0 0 1</diffuse>
+      <emissive>0 1 0 1</emissive>
+    </material>
+    <transparency>0.6</transparency>
+  </visual>
+  <!-- Inertia -->
+  <xacro:box_inertia
+    m="0.05"
+    x="0.015"
+    y="0.02"
+    z="0.03"
+    o_xyz="0 0 0"
+    o_rpy="0 0 0"/>
+</link>
+<joint name="l_ear_joint" type="revolute">
+  <parent link="base_link"/>
+  <child link="l_ear_link"/>
+  <origin xyz="0.165 0.04 0.74" rpy="0.0 0.25 0.0"/>
+  <axis xyz="0 0 1"/>
+  <limit lower="-0.2" upper="0.6" effort="0.1" velocity="10"/>
+  <dynamics friction="0.1" damping="0.1"/>
+</joint>
+<!-- ******************** RIGHT EAR ****************************** -->
+<link name="r_ear_link">
+  <visual name="r_ear_visual">
+    <origin xyz="0 0 0" rpy="0 0 0"/>
+    <geometry>
+      <box size="0.015 0.02 0.03"/>
+    </geometry>
+    <material name="k9_ear_emissive">
+      <ambient>0 0 0 1</ambient>
+      <diffuse>0 0 0 1</diffuse>
+      <emissive>0 0 0 1</emissive>
+    </material>
+  </visual>
+  <visual name="r_ear_beam_visual">
+    <origin xyz="1.0 0 0" rpy="0 0 0"/>
+    <geometry>
+      <cone radius="0.01" length="2.0"/>
+    </geometry>
+    <material name="k9_beam_material">
+      <ambient>0 0 0 1</ambient>
+      <diffuse>0 0 0 1</diffuse>
+      <emissive>0 1 0 1</emissive>
+    </material>
+    <transparency>0.6</transparency>
+  </visual>
+  <xacro:box_inertia
+    m="0.05"
+    x="0.015"
+    y="0.02"
+    z="0.03"
+    o_xyz="0 0 0"
+    o_rpy="0 0 0"/>
+</link>
+<joint name="r_ear_joint" type="revolute">
+  <parent link="base_link"/>
+  <child link="r_ear_link"/>
+  <origin xyz="0.165 -0.04 0.74" rpy="0.0 0.25 0.0"/>
+  <axis xyz="0 0 1"/>
+  <limit lower="-0.6" upper="0.2" effort="0.1" velocity="10"/>
+  <dynamics friction="0.1" damping="0.1"/>
+</joint>
   <!-- ===================================================== -->
   <!-- Gazebo Diff Drive (gz-sim, Jazzy)                     -->

Commit message: Update k9.urdf.xacro

File: src/k9_robot/src/description/k9.urdf.xacro (robot description, xacro)
@@ -228,13 +228,4 @@
           <cylinder radius="${wheel_radius}" length="${wheel_width}"/>
         </geometry>
-        <!-- NEW: slightly reduced friction to reduce "trip" under hard braking -->
-        <surface>
-          <friction>
-            <ode>
-              <mu>0.9</mu>
-              <mu2>0.7</mu2>
-            </ode>
-          </friction>
-        </surface>
       </collision>
       <inertial>
@@ -246,4 +237,8 @@
       </inertial>
     </link>
+    <gazebo reference="${name}_link">
+      <mu1>0.9</mu1>
+      <mu2>0.7</mu2>
+    </gazebo>
     <joint name="${name}_joint" type="continuous">
       <parent link="base_link"/>
@@ -270,16 +265,11 @@
         <sphere radius="${ball_radius}"/>
       </geometry>
-      <!-- NEW: low friction so it supports but doesn't brake/steer the robot -->
-      <surface>
-        <friction>
-          <ode>
-            <mu>0.2</mu>
-            <mu2>0.2</mu2>
-          </ode>
-        </friction>
-      </surface>
     </collision>
     <xacro:tiny_inertial m="0.5"/>
   </link>
+  <gazebo reference="ball_caster_link">
+    <mu1>0.2</mu1>
+    <mu2>0.2</mu2>
+  </gazebo>
   <joint name="ball_caster_joint" type="fixed">
     <parent link="base_link"/>
@@ -301,5 +291,5 @@
       <update_rate>10</update_rate>
       <always_on>true</always_on>
-      <topic>/world/empty/model/k9_robot/ld06/scan</topic>
+      <topic>/ld06/scan</topic>
       <pose>0 0 0 0 0 0</pose>
       <visualize>true</visualize>
@@ -346,5 +336,5 @@
   </visual>
   <visual name="l_ear_beam_visual">
-    <origin xyz="1.0 0 0" rpy="0 ${pi/2} 0"/>
+    <origin xyz="1.0075 0 0" rpy="0 ${pi/2} 0"/>
     <geometry>
       <cylinder radius="0.01" length="2.0"/>
@@ -360,4 +350,28 @@
   <xacro:tiny_inertial m="0.05"/>
 </link>
+<gazebo reference="l_ear_link">
+  <sensor name="l_ear_tof" type="ray">
+    <pose>0.0075 0 0 0 0 0</pose>
+    <update_rate>30</update_rate>
+    <always_on>true</always_on>
+    <visualize>true</visualize>
+    <topic>/l_ear/scan</topic>
+    <ray>
+      <scan>
+        <horizontal>
+          <samples>1</samples>
+          <resolution>1</resolution>
+          <min_angle>0</min_angle>
+          <max_angle>0</max_angle>
+        </horizontal>
+      </scan>
+      <range>
+        <min>0.02</min>
+        <max>2.0</max>
+        <resolution>0.001</resolution>
+      </range>
+    </ray>
+  </sensor>
+</gazebo>
 <joint name="l_ear_joint" type="revolute">
   <parent link="base_link"/>
@@ -382,5 +396,5 @@
   </visual>
   <visual name="r_ear_beam_visual">
-    <origin xyz="1.0 0 0" rpy="0 ${pi/2} 0"/>
+    <origin xyz="1.0075 0 0" rpy="0 ${pi/2} 0"/>
     <geometry>
       <cylinder radius="0.01" length="2.0"/>
@@ -395,4 +409,28 @@
   <xacro:tiny_inertial m="0.05"/>
 </link>
+<gazebo reference="r_ear_link">
+  <sensor name="r_ear_tof" type="ray">
+    <pose>0.0075 0 0 0 0 0</pose>
+    <update_rate>30</update_rate>
+    <always_on>true</always_on>
+    <visualize>true</visualize>
+    <topic>/r_ear/scan</topic>
+    <ray>
+      <scan>
+        <horizontal>
+          <samples>1</samples>
+          <resolution>1</resolution>
+          <min_angle>0</min_angle>
+          <max_angle>0</max_angle>
+        </horizontal>
+      </scan>
+      <range>
+        <min>0.02</min>
+        <max>2.0</max>
+        <resolution>0.001</resolution>
+      </range>
+    </ray>
+  </sensor>
+</gazebo>
 <joint name="r_ear_joint" type="revolute">
   <parent link="base_link"/>
@@ -403,4 +441,5 @@
   <dynamics friction="0.1" damping="0.1"/>
 </joint>
+<<<<<<< Updated upstream
 <xacro:k9_add_imu parent_link="base_link"
                   imu_link="imu_link"
@@ -410,4 +449,6 @@
                   accel_noise="0.01"
                   gyro_noise="0.001"/>
+=======
+>>>>>>> Stashed changes
   <!-- ===================================================== -->
   <!-- Gazebo Diff Drive (gz-sim, Jazzy)                     -->

Commit message: Add controller

File: src/k9_robot/src/description/k9.urdf.xacro (robot description, xacro)
@@ -471,4 +471,25 @@
     <dynamics friction="0.1" damping="0.1"/>
   </joint>
+  <!-- ===================================================== -->
+  <!-- Ear Joint Movement (gz-sim, Jazzy)                    -->
+  <!-- ===================================================== -->
+  <ros2_control name="K9EarsSystem" type="system">
+    <hardware>
+      <plugin>gz_ros2_control/GazeboSimSystem</plugin>
+    </hardware>
+    <joint name="l_ear_joint">
+      <command_interface name="position"/>
+      <state_interface name="position"/>
+      <state_interface name="velocity"/>
+    </joint>
+    <joint name="r_ear_joint">
+      <command_interface name="position"/>
+      <state_interface name="position"/>
+      <state_interface name="velocity"/>
+    </joint>
+  </ros2_control>
+  <!-- ===================================================== -->
+  <!-- IMU (gz-sim, Jazzy)                                   -->
+  <!-- ===================================================== -->
   <xacro:k9_add_imu
     parent_link="base_link"
@@ -506,4 +527,9 @@
       <child_frame_id>base_footprint</child_frame_id>
     </plugin>
-  </gazebo>
+  </gazebo><gazebo>
+  <plugin name="gz_ros2_control" filename="libgz_ros2_control-system.so">
+    <!-- Path inside your package is better than an absolute path -->
+    <parameters>/home/hopkira/Documents/GitHub/k9-gazebo/src/k9_robot/src/description/ears_controllers.yaml</parameters>
+  </plugin>
+</gazebo>
 </robot>

Commit message: Camera angle change

File: src/k9_robot/src/description/k9.urdf.xacro (robot description, xacro)
@@ -171,5 +171,5 @@
       <parent link="oakd_link"/>   <!-- or oakd_link / 3dcam_link, whichever is your camera body -->
       <child  link="camera_depth_frame"/>
-      <origin xyz="0 0 0" rpy="0 0 0"/>
+      <origin xyz="0 0 0" rpy="${-pi/2} 0 ${-pi/2}"/>
     </joint>
     <gazebo reference="${oak_link}">
