Commit message: Make K9 model portable and unify Jazzy simulation bring-up

File: src/k9_robot/src/description/k9.urdf.xacro (robot description, xacro)
@@ -1,9 +1,11 @@
 <?xml version="1.0"?>
 <robot name="k9_robot" xmlns:xacro="http://ros.org/wiki/xacro">
+  <xacro:arg name="description_share" default="$(find k9_description)"/>
+  <xacro:arg name="controllers_file" default="$(find k9_description)/config/controllers.yaml"/>
+  <xacro:arg name="sim" default="true"/>
   <!-- ===================================================== -->
   <!-- To generate SDF for Gazebo Sim                        -->
-  <!-- ros2 run xacro xacro k9.urdf.xacro > k9.urdf          -->
-  <!-- gz sdf -p k9.urdf > k9_raw.sdf                        -->
-  <!-- python3 patch_friction.py k9_raw.sdf k9_robot.sdf     -->
+  <!-- Source the built workspace, then run gen.sh.          -->
+  <!-- Exports are generated outside the source tree.        -->
   <!-- ===================================================== -->
   <!-- ===================================================== -->
@@ -42,4 +44,12 @@
         iyy="1e-4" iyz="0"
         izz="1e-4"/>
+    </inertial>
+  </xacro:macro>
+  <!-- Uniform-density approximations; dimensions are in metres. -->
+  <xacro:macro name="box_inertial" params="m x y z">
+    <inertial>
+      <mass value="${m}"/>
+      <inertia ixx="${m*(y*y+z*z)/12}" iyy="${m*(x*x+z*z)/12}"
+               izz="${m*(x*x+y*y)/12}" ixy="0" ixz="0" iyz="0"/>
     </inertial>
   </xacro:macro>
@@ -75,4 +85,5 @@
       <sensor name="${imu_link}_sensor" type="imu">
         <topic>/k9/imu</topic>
+        <gz_frame_id>${imu_link}</gz_frame_id>
         <always_on>true</always_on>
         <visualize>false</visualize>
@@ -179,4 +190,5 @@
         <update_rate>${update_rate}</update_rate>
         <topic>${gz_topic}</topic>
+        <gz_frame_id>${frame_id}</gz_frame_id>
         <camera>
           <horizontal_fov>${hfov}</horizontal_fov>
@@ -210,15 +222,21 @@
       <origin xyz="-0.5 1.905 ${-wheel_radius}" rpy="0 0 ${pi}"/>
       <geometry>
-        <mesh filename="file:///home/hopkira/Documents/GitHub/k9-gazebo/src/k9_description/urdf/k9.stl"
+        <mesh filename="file://$(arg description_share)/urdf/k9.stl"
               scale="0.01 0.01 0.01"/>
       </geometry>
       <material name="K9_grey"/>
     </visual>
-    <!-- Collision -->
-    <collision>
-      <origin xyz="0.0 0.0 0.44"/>
-      <geometry>
-        <box size="1.05 0.49 0.74"/>
-      </geometry>
+    <!-- Conservative body / head envelopes fitted to k9.stl.
+         Heights below are measured from the ground, then shifted into base_link.
+         The body includes the skirt and back-panel fittings; the head includes
+         ears. Boxes intentionally approximate the sloping shell (see docs/PHYSICS.md).
+         Default self-collision remains off: wheels sit inside the body envelope. -->
+    <collision name="body_collision">
+      <origin xyz="-0.1175 0 ${0.29-wheel_radius}"/>
+      <geometry><box size="0.815 0.49 0.50"/></geometry>
+    </collision>
+    <collision name="head_collision">
+      <origin xyz="0.329 0 ${0.6275-wheel_radius}"/>
+      <geometry><box size="0.404 0.174 0.265"/></geometry>
     </collision>
     <!-- Inertia: main shell + structure -->
@@ -250,5 +268,5 @@
       </geometry>
     </collision>
-    <xacro:tiny_inertial m="5.0"/>
+    <xacro:box_inertial m="5.0" x="0.25" y="0.20" z="0.25"/>
   </link>
   <joint name="battery_joint" type="fixed">
@@ -266,5 +284,5 @@
       </geometry>
     </collision>
-    <xacro:tiny_inertial m="3.0"/>
+    <xacro:box_inertial m="3.0" x="0.20" y="0.20" z="0.10"/>
   </link>
   <joint name="motors_joint" type="fixed">
@@ -291,15 +309,16 @@
         </geometry>
       </collision>
+      <!-- Solid 1 kg cylinder; its axle is Y in the link frame. -->
       <inertial>
         <mass value="1.0"/>
         <inertia
-          ixx="0.002" ixy="0" ixz="0"
-          iyy="0.002" iyz="0"
-          izz="0.004"/>
+          ixx="${(3*wheel_radius*wheel_radius+wheel_width*wheel_width)/12}" ixy="0" ixz="0"
+          iyy="${wheel_radius*wheel_radius/2}" iyz="0"
+          izz="${(3*wheel_radius*wheel_radius+wheel_width*wheel_width)/12}"/>
       </inertial>
     </link>
     <gazebo reference="${name}_link">
-      <mu1>0.9</mu1>
-      <mu2>0.7</mu2>
+      <mu1>1.1</mu1>
+      <mu2>0.9</mu2>
     </gazebo>
     <joint name="${name}_joint" type="continuous">
@@ -328,5 +347,10 @@
       </geometry>
     </collision>
-    <xacro:tiny_inertial m="0.5"/>
+    <inertial>
+      <mass value="0.5"/>
+      <inertia ixx="${2*0.5*ball_radius*ball_radius/5}"
+               iyy="${2*0.5*ball_radius*ball_radius/5}"
+               izz="${2*0.5*ball_radius*ball_radius/5}" ixy="0" ixz="0" iyz="0"/>
+    </inertial>
   </link>
   <gazebo reference="ball_caster_link">
@@ -334,4 +358,10 @@
     <mu2>0.2</mu2>
   </gazebo>
+  <!-- URDF has no spherical joint. Keep this nominal frame for ROS; the shared
+       SDF export step replaces this preserved joint with a native passive ball
+       joint. A sphere has no meaningful visual orientation and carries no sensor. -->
+  <gazebo reference="ball_caster_joint">
+    <preserveFixedJoint>true</preserveFixedJoint>
+  </gazebo>
   <joint name="ball_caster_joint" type="fixed">
     <parent link="base_link"/>
@@ -342,5 +372,5 @@
   <!-- Sensors                                               -->
   <!-- ===================================================== -->
-  <!-- started at 0.565 raised by 20 cm to clear body       -->
+  <!-- Back-panel lidar intentionally sees the head in its forward sector. -->
   <link name="base_laser"><xacro:tiny_inertial m="0.05"/></link>
   <joint name="base_laser_joint" type="fixed">
@@ -401,13 +431,20 @@
     <xacro:tiny_inertial m="0.05"/>
   </link>
+  <!-- Sensor mount is 30 degrees below the rotating ear; servo axis tilts 7 degrees. -->
+  <link name="l_ear_sensor_link"/>
+  <joint name="l_ear_sensor_joint" type="fixed">
+    <parent link="l_ear_link"/>
+    <child link="l_ear_sensor_link"/>
+    <origin xyz="0.0075 0 0" rpy="0 ${pi/6} 0"/>
+  </joint>
   <gazebo reference="l_ear_link">
     <sensor name="l_ear_tof" type="gpu_lidar">
-      <pose>0.0075 0 0 0 0 0</pose>
+      <pose>0.0075 0 0 0 ${pi/6} 0</pose>
       <update_rate>30</update_rate>
       <always_on>true</always_on>
       <visualize>true</visualize>
       <topic>/l_ear/scan</topic>
-      <gz_frame_id>l_ear_link</gz_frame_id>
-      <frame_id>l_ear_link</frame_id>
+      <gz_frame_id>l_ear_sensor_link</gz_frame_id>
+      <frame_id>l_ear_sensor_link</frame_id>
       <lidar>
         <scan>
@@ -430,5 +467,5 @@
     <parent link="base_link"/>
     <child link="l_ear_link"/>
-    <origin xyz="0.27 0.0425 0.67" rpy="0.0 0.25 0.0"/>
+    <origin xyz="0.27 0.0425 0.67" rpy="0 ${7*pi/180} 0"/>
     <axis xyz="0 0 1"/>
     <limit lower="-0.2" upper="0.6" effort="2.0" velocity="10"/>
@@ -450,13 +487,20 @@
     <xacro:tiny_inertial m="0.05"/>
   </link>
+  <!-- Sensor mount is 30 degrees below the rotating ear; servo axis tilts 7 degrees. -->
+  <link name="r_ear_sensor_link"/>
+  <joint name="r_ear_sensor_joint" type="fixed">
+    <parent link="r_ear_link"/>
+    <child link="r_ear_sensor_link"/>
+    <origin xyz="0.0075 0 0" rpy="0 ${pi/6} 0"/>
+  </joint>
   <gazebo reference="r_ear_link">
     <sensor name="r_ear_tof" type="gpu_lidar">
-      <pose>0.0075 0 0 0 0 0</pose>
+      <pose>0.0075 0 0 0 ${pi/6} 0</pose>
       <update_rate>30</update_rate>
       <always_on>true</always_on>
       <visualize>true</visualize>
       <topic>/r_ear/scan</topic>
-      <gz_frame_id>r_ear_link</gz_frame_id>
-      <frame_id>r_ear_link</frame_id>
+      <gz_frame_id>r_ear_sensor_link</gz_frame_id>
+      <frame_id>r_ear_sensor_link</frame_id>
       <lidar>
         <scan>
@@ -479,5 +523,5 @@
     <parent link="base_link"/>
     <child link="r_ear_link"/>
-    <origin xyz="0.27 -0.0425 0.67" rpy="0.0 0.25 0.0"/>
+    <origin xyz="0.27 -0.0425 0.67" rpy="0 ${7*pi/180} 0"/>
     <axis xyz="0 0 1"/>
     <limit lower="-0.6" upper="0.2" effort="2.0" velocity="10"/>
@@ -485,21 +529,33 @@
   </joint>
   <!-- ===================================================== -->
-  <!-- Ear Joint Movement (gz-sim, Jazzy)                    -->
-  <!-- ===================================================== -->
-  <ros2_control name="K9EarsSystem" type="system">
-    <hardware>
-      <plugin>gz_ros2_control/GazeboSimSystem</plugin>
-    </hardware>
-    <joint name="l_ear_joint">
-      <command_interface name="position"/>
-      <state_interface name="position"/>
-      <state_interface name="velocity"/>
-    </joint>
-    <joint name="r_ear_joint">
-      <command_interface name="position"/>
-      <state_interface name="position"/>
-      <state_interface name="velocity"/>
-    </joint>
-  </ros2_control>
+  <!-- Wheel and ear joint control (gz-sim, Jazzy)            -->
+  <!-- ===================================================== -->
+  <xacro:if value="$(arg sim)">
+    <ros2_control name="K9SimSystem" type="system">
+      <hardware>
+        <plugin>gz_ros2_control/GazeboSimSystem</plugin>
+      </hardware>
+      <joint name="drivewhl_l_joint">
+        <command_interface name="velocity"/>
+        <state_interface name="position"/>
+        <state_interface name="velocity"/>
+      </joint>
+      <joint name="drivewhl_r_joint">
+        <command_interface name="velocity"/>
+        <state_interface name="position"/>
+        <state_interface name="velocity"/>
+      </joint>
+      <joint name="l_ear_joint">
+        <command_interface name="position"/>
+        <state_interface name="position"/>
+        <state_interface name="velocity"/>
+      </joint>
+      <joint name="r_ear_joint">
+        <command_interface name="position"/>
+        <state_interface name="position"/>
+        <state_interface name="velocity"/>
+      </joint>
+    </ros2_control>
+  </xacro:if>
   <!-- ===================================================== -->
   <!-- IMU (gz-sim, Jazzy)                                   -->
@@ -519,32 +575,13 @@
     rpy="0 0 0"
     gz_topic="/oak"
-    frame_id="oak_depth_frame"/>
-  <!-- ===================================================== -->
-  <!-- Gazebo Diff Drive (gz-sim, Jazzy)                     -->
-  <!-- ===================================================== -->
-  <gazebo>
-    <plugin filename="gz-sim-diff-drive-system"
-            name="gz::sim::systems::DiffDrive">
-      <left_joint>drivewhl_l_joint</left_joint>
-      <right_joint>drivewhl_r_joint</right_joint>
-      <wheel_separation>${track}</wheel_separation>
-      <wheel_radius>${wheel_radius}</wheel_radius>
-      <max_linear_velocity>1.4</max_linear_velocity>
-      <max_angular_velocity>0.63</max_angular_velocity>
-      <!-- CHANGED: lower accel also caps braking decel (less "nose dive") -->
-      <max_linear_acceleration>0.28</max_linear_acceleration>
-      <max_angular_acceleration>0.21</max_angular_acceleration>
-      <topic>/cmd_vel_nav</topic>
-      <odom_topic>/odom</odom_topic>
-      <odom_publish_frequency>50</odom_publish_frequency>
-       <tf_topic>/tf</tf_topic>
-      <frame_id>odom</frame_id>
-      <child_frame_id>base_footprint</child_frame_id>
-    </plugin>
-  </gazebo>
-  <gazebo>
-    <plugin name="gz_ros2_control::GazeboSimROS2ControlPlugin" filename="/opt/ros/jazzy/lib/libgz_ros2_control-system.so">
-      <parameters>/home/hopkira/Documents/GitHub/k9-gazebo/src/k9_robot/src/description/ear_controllers.yaml</parameters>
-    </plugin>
-  </gazebo>
+    frame_id="camera_depth_frame"/>
+  <!-- One controller manager owns wheel and ear command interfaces. -->
+  <xacro:if value="$(arg sim)">
+    <gazebo>
+      <plugin name="gz_ros2_control::GazeboSimROS2ControlPlugin"
+              filename="libgz_ros2_control-system.so">
+        <parameters>$(arg controllers_file)</parameters>
+      </plugin>
+    </gazebo>
+  </xacro:if>
 </robot>

Commit message: Adding motors and latest nav config

File: src/k9_robot/src/description/k9.urdf.xacro (robot description, xacro)
@@ -29,5 +29,42 @@
   <xacro:property name="wheel_radius" value="0.0694"/>
   <xacro:property name="wheel_width"  value="0.025"/>
-  <xacro:property name="track"         value="0.2022"/>
+  <xacro:property name="track"        value="0.2022"/>
+  <!-- ===================================================== -->
+  <!-- Drive transmission and motor model                    -->
+  <!--                                                       -->
+  <!-- MY6812 brushed motors, supplied at 27.68 V.           -->
+  <!-- 16-tooth motor pulley to 88-tooth wheel pulley.       -->
+  <!-- Motor constants and rotor inertia remain provisional  -->
+  <!-- until measured on K9's actual motors.                 -->
+  <!-- ===================================================== -->
+  <xacro:property name="motor_pulley_teeth" value="16.0"/>
+  <xacro:property name="wheel_pulley_teeth" value="88.0"/>
+  <xacro:property name="drive_reduction"
+                  value="${wheel_pulley_teeth / motor_pulley_teeth}"/>
+  <xacro:property name="motor_supply_voltage" value="27.68"/>
+  <xacro:property name="motor_back_emf_constant" value="0.082"/>
+  <xacro:property name="motor_torque_constant" value="0.082"/>
+  <xacro:property name="motor_current_limit" value="15.0"/>
+  <xacro:property name="belt_efficiency" value="0.90"/>
+  <!-- Theoretical no-load speeds: approximately 337.6 rad/s
+       at the motor and 61.4 rad/s at the wheel. -->
+  <xacro:property name="motor_no_load_speed"
+                  value="${motor_supply_voltage / motor_back_emf_constant}"/>
+  <xacro:property name="wheel_max_speed"
+                  value="${motor_no_load_speed / drive_reduction}"/>
+  <!-- Short-duration wheel effort at the RoboClaw's 15 A
+       per-channel current limit: approximately 6.09 N m. -->
+  <xacro:property name="wheel_max_effort"
+                  value="${motor_torque_constant
+                           * motor_current_limit
+                           * drive_reduction
+                           * belt_efficiency}"/>
+  <!-- Estimated motor inertia reflected to the wheel shaft:
+       0.00003 * 5.5^2 = 0.0009075 kg m^2. -->
+  <xacro:property name="motor_rotor_inertia" value="0.00003"/>
+  <xacro:property name="reflected_motor_inertia"
+                  value="${motor_rotor_inertia
+                           * drive_reduction
+                           * drive_reduction}"/>
   <!-- Ball caster -->
   <xacro:property name="ball_radius"  value="0.04"/>
@@ -178,8 +215,8 @@
     </joint>
     <!-- Depth frame used by Gazebo / depthimage_to_laserscan -->
-    <link name="camera_depth_frame"/>
-    <joint name="camera_depth_frame_joint" type="fixed">
-      <parent link="oakd_link"/>   <!-- or oakd_link / 3dcam_link, whichever is your camera body -->
-      <child  link="camera_depth_frame"/>
+    <link name="oak_rgb_camera_optical_frame"/>
+    <joint name="oak_rgb_camera_optical_frame_joint" type="fixed">
+      <parent link="${oak_link}"/>
+      <child link="oak_rgb_camera_optical_frame"/>
       <origin xyz="0 0 0" rpy="${-pi/2} 0 ${-pi/2}"/>
     </joint>
@@ -309,10 +346,11 @@
         </geometry>
       </collision>
-      <!-- Solid 1 kg cylinder; its axle is Y in the link frame. -->
+      <!-- Solid 1 kg cylinder plus motor inertia reflected through
+           the 5.5:1 belt reduction; axle is Y in the link frame. -->
       <inertial>
         <mass value="1.0"/>
         <inertia
           ixx="${(3*wheel_radius*wheel_radius+wheel_width*wheel_width)/12}" ixy="0" ixz="0"
-          iyy="${wheel_radius*wheel_radius/2}" iyz="0"
+          iyy="${wheel_radius*wheel_radius/2 + reflected_motor_inertia}" iyz="0"
           izz="${(3*wheel_radius*wheel_radius+wheel_width*wheel_width)/12}"/>
       </inertial>
@@ -327,5 +365,9 @@
       <origin xyz="0 ${y} 0"/>
       <axis xyz="0 1 0"/>
-      <dynamics damping="0.05"/>
+      <!-- Wheel-side limits derived from the motor, 27.68 V supply,
+           5.5:1 belt reduction and 15 A controller current limit. -->
+      <limit effort="${wheel_max_effort}"
+             velocity="${wheel_max_speed}"/>
+      <dynamics damping="0.02" friction="0.04"/>
     </joint>
   </xacro:macro>
@@ -537,12 +579,20 @@
       </hardware>
       <joint name="drivewhl_l_joint">
-        <command_interface name="velocity"/>
+        <command_interface name="velocity">
+          <param name="min">${-wheel_max_speed}</param>
+          <param name="max">${wheel_max_speed}</param>
+        </command_interface>
         <state_interface name="position"/>
         <state_interface name="velocity"/>
+        <state_interface name="effort"/>
       </joint>
       <joint name="drivewhl_r_joint">
-        <command_interface name="velocity"/>
+        <command_interface name="velocity">
+          <param name="min">${-wheel_max_speed}</param>
+          <param name="max">${wheel_max_speed}</param>
+        </command_interface>
         <state_interface name="position"/>
         <state_interface name="velocity"/>
+        <state_interface name="effort"/>
       </joint>
       <joint name="l_ear_joint">
@@ -575,5 +625,5 @@
     rpy="0 0 0"
     gz_topic="/oak"
-    frame_id="camera_depth_frame"/>
+    frame_id="oak_rgb_camera_optical_frame"/>
   <!-- One controller manager owns wheel and ear command interfaces. -->
   <xacro:if value="$(arg sim)">
