Commit message: Initial build

File: src/k9_robot/src/description/k9.urdf (robot description, URDF)
Before this commit: robot k9_robot, 6 links, 5 joints
Links:
- link base_link: geometry collision box size=${base_length} ${base_width} ${base_height}; collision box size=0.43 0.18 0.295

Commit message: Update k9.urdf

File: src/k9_robot/src/description/k9.urdf (robot description, URDF)
Before this commit: robot k9_robot, 6 links, 5 joints
Joints:
- joint 3dcam_joint: origin xyz=0.206 0.0 -0.042 rpy=0 0 0 -> xyz=0.206 0.0 0.255 rpy=0 0 0
- joint caster_joint: origin xyz=${caster_xoff} 0.0 ${-(caster_z_offset)} rpy=0 0 0 -> xyz=${caster_xoff} 0.0 ${caster_z_offset} rpy=0 0 0
- joint eyecam_joint: origin xyz=0.366 0.0 0.373 rpy=0 0 0 -> xyz=0.366 0.0 0.67 rpy=0 0 0
- joint lidar_joint: origin xyz=-0.112 0.0 0.268 rpy=0 0 0 -> xyz=-0.112 0.0 0.565 rpy=0 0 0

Commit message: Update k9.urdf

File: src/k9_robot/src/description/k9.urdf (robot description, URDF)
Before this commit: robot k9_robot, 6 links, 5 joints
Joints:
- joint base_joint: origin xyz=0.0 0.0 ${(wheel_radius-wheel_zoff)} rpy=0 0 0 -> xyz=0.0 0.0 ${-(wheel_radius)} rpy=0 0 0

Commit message: Screenshot and working version

File: src/k9_robot/src/description/k9.urdf (robot description, URDF)
Before this commit: robot k9_robot, 6 links, 5 joints
Joints:
- joint base_joint: origin xyz=0.0 0.0 ${-(wheel_radius)} rpy=0 0 0 -> xyz=0.0 0.0 0.0 rpy=0 0 0
- joint caster_joint: origin xyz=${caster_xoff} 0.0 ${caster_z_offset} rpy=0 0 0 -> xyz=${caster_xoff} 0.0 ${-(caster_z_offset)} rpy=0 0 0

Commit message: Added ears

File: src/k9_robot/src/description/k9.urdf (robot description, URDF)
Before this commit: robot k9_robot, 6 links, 5 joints
Links:
- added link l_ear_link
- added link r_ear_link
Joints:
- added joint l_ear_joint: type fixed, parent base_link, child l_ear_link, origin xyz=0.35 -0.045 0.725 rpy=0 -0.65 0
- added joint r_ear_joint: type fixed, parent base_link, child r_ear_link, origin xyz=0.35 0.045 0.725 rpy=0 -0.65 0

Commit message: Change castor details

File: src/k9_robot/src/description/k9.urdf (robot description, URDF)
Before this commit: robot k9_robot, 8 links, 7 joints
Links:
- removed link front_caster
- added link rear_castor; collision sphere radius=0.02; visual sphere radius=0.02
Joints:
- removed joint caster_joint
- added joint castor_joint: type fixed, parent base_link, child rear_castor, origin xyz=${castor_xoff} 0.0 ${-(castor_z_offset)} rpy=0 0 0

Commit message: Update k9.urdf

File: src/k9_robot/src/description/k9.urdf (robot description, URDF)
Before this commit: robot k9_robot, 8 links, 7 joints
Links:
- link base_link: geometry collision box size=0.43 0.18 0.295; collision box size=0.89 0.49 0.52
Joints:
- joint 3dcam_joint: origin xyz=0.206 0.0 0.255 rpy=0 0 0 -> xyz=0.206 0.0 0.255 rpy=0.0 0.0 0.0
- joint castor_joint: origin xyz=${castor_xoff} 0.0 ${-(castor_z_offset)} rpy=0 0 0 -> xyz=-0.298 0.0 0.02 rpy=0 0 0
- joint eyecam_joint: origin xyz=0.366 0.0 0.67 rpy=0 0 0 -> xyz=0.366 0.0 0.67 rpy=0.0 0.0 0.0
- joint l_ear_joint: origin xyz=0.35 -0.045 0.725 rpy=0 -0.65 0 -> xyz=0.35 0.045 0.725 rpy=0.0 0.65 0.0
- joint lidar_joint: origin xyz=-0.112 0.0 0.565 rpy=0 0 0 -> xyz=-0.112 0.0 0.565 rpy=0.0 0.0 0.0
- joint r_ear_joint: origin xyz=0.35 0.045 0.725 rpy=0 -0.65 0 -> xyz=0.35 -0.045 0.725 rpy=0.0 0.65 0.0

Commit message: Expert walkthrough by LLM

File: src/k9_robot/src/description/k9.urdf (robot description, URDF)
Before this commit: robot k9_robot, 8 links, 7 joints
Links:
- removed link rear_castor
- added link caster_swivel_link; collision cylinder length=0.03 radius=0.008; visual cylinder length=0.03 radius=0.008
- added link caster_wheel_link; collision cylinder length=${caster_wheel_width} radius=${caster_wheel_radius}; visual cylinder length=${caster_wheel_width} radius=${caster_wheel_radius}
- link base_link: mass None -> 27.0; geometry collision box size=0.43 0.18 0.295; collision box size=0.89 0.49 0.35
Joints:
- removed joint castor_joint
- added joint caster_swivel_joint: type continuous, parent base_link, child caster_swivel_link, origin xyz=${caster_mount_x} ${caster_mount_y} ${caster_mount_z} rpy=0 0 0, axis 0 0 1
- added joint caster_wheel_joint: type continuous, parent caster_swivel_link, child caster_wheel_link, origin xyz=${-caster_fork_offset} 0 0 rpy=0 0 0, axis 0 1 0
- joint base_joint: child base_footprint -> base_link; origin xyz=0.0 0.0 0.0 rpy=0 0 0 -> xyz=0.0 0.0 ${wheel_radius} rpy=0 0 0; parent base_link -> base_footprint

Commit message: Fixing URDF Significant update done on Ubuntu gazebo machine

File: src/k9_robot/src/description/k9.urdf (robot description, URDF)
Before this commit: robot k9_robot, 11 links, 10 joints
Links:
- removed link caster_swivel_link
- removed link caster_wheel_link
- removed link l_ear_link
- removed link lidar_link
- removed link r_ear_link
- added link ball_caster_link, mass 0.5; collision sphere radius=0.04; visual sphere radius=0.04
- added link base_laser, mass 0.05
- added link battery_link, mass 5.0; collision box size=0.25 0.20 0.25
- added link motors_link, mass 3.0; collision box size=0.20 0.20 0.10
- link base_link: mass 25.0 -> 19.0; geometry collision box size=1.05 0.49 0.74; visual mesh filename=file:///home/hopkira/Documents/GitHub/k9-gazebo/src/k9_desc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 scale=0.01 0.01 0.01
- link drivewhl_l_link: geometry collision cylinder length=0.025 radius=0.0694; visual cylinder length=0.025 radius=0.0694
- link drivewhl_r_link: geometry collision cylinder length=0.025 radius=0.0694; visual cylinder length=0.025 radius=0.0694
Joints:
- removed joint caster_swivel_joint
- removed joint caster_wheel_joint
- removed joint l_ear_joint
- removed joint lidar_joint
- removed joint r_ear_joint
- added joint ball_caster_joint: type fixed, parent base_link, child ball_caster_link, origin xyz=-0.3 0 -0.029400000000000003
- added joint base_laser_joint: type fixed, parent base_link, child base_laser, origin xyz=-0.112 0 0.53 rpy=0 0 0
- added joint battery_joint: type fixed, parent base_link, child battery_link, origin xyz=0 0 0.18
- added joint motors_joint: type fixed, parent base_link, child motors_link, origin xyz=0 0 0.10
- joint 3dcam_joint: origin xyz=0.206 0.0 0.255 rpy=0.0 0.0 0.0 -> xyz=0.206 0 0.255
- joint base_joint: origin xyz=0.0 0.0 0.06939 rpy=0 0 0 -> xyz=0 0 0.0694
- joint drivewhl_l_joint: origin xyz=0.0 0.1011 0.06939 rpy=0 0 0 -> xyz=0 0.1011 0; parent base_footprint -> base_link
- joint drivewhl_r_joint: origin xyz=0.0 -0.1011 0.06939 rpy=0 0 0 -> xyz=0 -0.1011 0; parent base_footprint -> base_link
- joint eyecam_joint: origin xyz=0.366 0.0 0.67 rpy=0.0 0.0 0.0 -> xyz=0.366 0 0.67

File: src/k9_robot/src/description/k9.urdf.xacro (robot description, xacro)
@@ -1,14 +1,21 @@
-<?xml version="1.0" ?>
+<?xml version="1.0"?>
 <robot name="k9_robot" xmlns:xacro="http://ros.org/wiki/xacro">
-  <!-- ===================== Materials ===================== -->
+  <!-- ===================================================== -->
+  <!-- Materials                                             -->
+  <!-- ===================================================== -->
   <material name="K9_grey">
+<<<<<<< HEAD
     <color rgba="0.25 0.25 0.25 1.0" />
   </material>
   <material name="perspex_red">
     <color rgba="1.0 0.1 0.1 1.0" />
+=======
+    <color rgba="0.25 0.25 0.25 1.0"/>
+>>>>>>> b2d86b1 (Fixing URDF)
   </material>
   <material name="wheel_grey">
     <color rgba="0.7 0.7 0.7 1.0"/>
   </material>
+<<<<<<< HEAD
   <material name="white">
     <color rgba="1.0 1.0 1.0 1.0"/>
@@ -22,30 +29,29 @@
   <!-- Drive wheels (m) -->
   <xacro:property name="wheel_radius" value="0.06939"/>
+=======
+  <!-- ===================================================== -->
+  <!-- Constants                                             -->
+  <!-- ===================================================== -->
+  <xacro:property name="wheel_radius" value="0.0694"/>
+>>>>>>> b2d86b1 (Fixing URDF)
   <xacro:property name="wheel_width"  value="0.025"/>
-  <!-- Wheel center-to-center separation (m) -->
-  <xacro:property name="track" value="0.2022"/>
-  <!-- Wheel x offset relative to base_link -->
-  <xacro:property name="wheel_xoff" value="0.0"/>
-  <!-- Caster configuration -->
-  <xacro:property name="castor_xoff" value="-0.298"/>
-  <!-- 40 mm caster wheel -->
-  <xacro:property name="caster_wheel_radius" value="0.02"/>
-  <xacro:property name="caster_wheel_width"  value="0.012"/>
-  <xacro:property name="caster_fork_offset"  value="0.018"/>  <!-- axle behind swivel -->
-  <xacro:property name="caster_mount_x" value="${castor_xoff}"/>
-  <xacro:property name="caster_mount_y" value="0.0"/>
-  <!-- base_link is at axle height; place swivel so wheel touches ground -->
-  <xacro:property name="caster_mount_z" value="${-wheel_radius + caster_wheel_radius -0.002}"/>
-  <!-- ===================== Inertia helper macros ===================== -->
-  <xacro:macro name="box_inertia" params="m w h d">
+  <xacro:property name="track"         value="0.2022"/>
+  <!-- Ball caster -->
+  <xacro:property name="ball_radius"  value="0.04"/>
+  <xacro:property name="ball_x"       value="-0.30"/>
+  <!-- ===================================================== -->
+  <!-- Helper macros                                         -->
+  <!-- ===================================================== -->
+  <xacro:macro name="tiny_inertial" params="m">
     <inertial>
-      <origin xyz="0 0 0" rpy="0 0 0"/>
+      <origin xyz="0 0 0"/>
       <mass value="${m}"/>
       <inertia
-        ixx="${(m/12) * (h*h + d*d)}" ixy="0.0" ixz="0.0"
-        iyy="${(m/12) * (w*w + d*d)}" iyz="0.0"
-        izz="${(m/12) * (w*w + h*h)}"/>
+        ixx="1e-4" ixy="0" ixz="0"
+        iyy="1e-4" iyz="0"
+        izz="1e-4"/>
     </inertial>
   </xacro:macro>
+<<<<<<< HEAD
   <!-- Cylinder inertia about its own center.
       rpy must match the cylinder geometry orientation -->
@@ -69,27 +75,34 @@
   </xacro:macro>
   <!-- ===================== Base frames ===================== -->
+=======
+  <!-- ===================================================== -->
+  <!-- Frames                                                -->
+  <!-- ===================================================== -->
+>>>>>>> b2d86b1 (Fixing URDF)
   <link name="base_footprint"/>
+  <!-- ===================================================== -->
+  <!-- Base / chassis                                        -->
+  <!-- ===================================================== -->
   <link name="base_link">
+    <!-- Visual -->
     <visual>
-      <origin xyz="-0.5 1.905 0" rpy="0 0 ${pi}"/>
-      <geometry>
-        <mesh filename="file:///home/hopkira/Documents/GitHub/k9-gazebo/src/k9_description/urdf/k9.stl" scale="0.01 0.01 0.01"/>
+      <origin xyz="-0.5 1.905 ${-wheel_radius}" rpy="0 0 ${pi}"/>
+      <geometry>
+        <mesh filename="file:///home/hopkira/Documents/GitHub/k9-gazebo/src/k9_description/urdf/k9.stl"
+              scale="0.01 0.01 0.01"/>
       </geometry>
       <material name="K9_grey"/>
     </visual>
-    <!-- Collision layout avoids wheels and mirrors head/body -->
-    <collision>
-      <origin xyz="-0.119 0.0 0.285" rpy="0.0 0.0 0.0"/>
-      <geometry>
-        <box size="0.89 0.49 0.49"/>
-      </geometry>
-    </collision>
-    <collision>
-      <origin xyz="0.336 0.0 0.6125" rpy="0.0 0.0 0.0"/>
-      <geometry>
-        <box size="0.43 0.18 0.295"/>
-      </geometry>
-    </collision>
+    <!-- Collision -->
+    <collision>
+      <origin xyz="0.0 0.0 0.44"/>
+      <geometry>
+        <box size="1.05 0.49 0.74"/>
+      </geometry>
+    </collision>
+    <!-- Inertia: main shell + structure -->
+    <!-- CHANGED: lower + slightly rear-shift COM, and increase pitch inertia (iyy) -->
     <inertial>
+<<<<<<< HEAD
       <!-- Recomputed from 5 internal mass boxes (total 25.0 kg).
           Origin is COM expressed in base_link frame. -->
@@ -100,4 +113,15 @@
         iyy="2.263333"  iyz="0.0"
         izz="1.639449"/>
+=======
+      <!-- was: -0.02 0 0.20 -->
+      <origin xyz="-0.06 0 0.16"/>
+      <mass value="19.0"/>
+      <inertia
+        ixx="0.80"
+        ixy="0" ixz="0"
+        iyy="2.40"
+        iyz="0"
+        izz="1.70"/>
+>>>>>>> b2d86b1 (Fixing URDF)
     </inertial>
   </link>
@@ -105,11 +129,45 @@
     <parent link="base_footprint"/>
     <child link="base_link"/>
-    <origin xyz="0.0 0.0 ${wheel_radius}" rpy="0 0 0"/>
-  </joint>
-  <!-- ===================== Drive wheels ===================== -->
-  <xacro:macro name="wheel" params="prefix x y">
-    <link name="${prefix}_link">
+    <origin xyz="0 0 ${wheel_radius}"/>
+  </joint>
+  <!-- ===================================================== -->
+  <!-- Battery (low + central)                               -->
+  <!-- ===================================================== -->
+  <link name="battery_link">
+    <collision>
+      <geometry>
+        <box size="0.25 0.20 0.25"/>
+      </geometry>
+    </collision>
+    <xacro:tiny_inertial m="5.0"/>
+  </link>
+  <joint name="battery_joint" type="fixed">
+    <parent link="base_link"/>
+    <child link="battery_link"/>
+    <origin xyz="0 0 0.18"/>
+  </joint>
+  <!-- ===================================================== -->
+  <!-- Motors                                                -->
+  <!-- ===================================================== -->
+  <link name="motors_link">
+    <collision>
+      <geometry>
+        <box size="0.20 0.20 0.10"/>
+      </geometry>
+    </collision>
+    <xacro:tiny_inertial m="3.0"/>
+  </link>
+  <joint name="motors_joint" type="fixed">
+    <parent link="base_link"/>
+    <child link="motors_link"/>
+    <origin xyz="0 0 0.10"/>
+  </joint>
+  <!-- ===================================================== -->
+  <!-- Drive wheels                                          -->
+  <!-- ===================================================== -->
+  <xacro:macro name="drive_wheel" params="name y">
+    <link name="${name}_link">
       <visual>
-        <origin xyz="0 0 0" rpy="${pi/2} 0 0"/>
+        <origin rpy="${pi/2} 0 0"/>
         <geometry>
           <cylinder radius="${wheel_radius}" length="${wheel_width}"/>
@@ -118,9 +176,19 @@
       </visual>
       <collision>
-        <origin xyz="0 0 0" rpy="${pi/2} 0 0"/>
+        <origin rpy="${pi/2} 0 0"/>
         <geometry>
           <cylinder radius="${wheel_radius}" length="${wheel_width}"/>
         </geometry>
+        <!-- NEW: slightly reduced friction to reduce "trip" under hard braking -->
+        <surface>
+          <friction>
+            <ode>
+              <mu>0.9</mu>
+              <mu2>0.7</mu2>
+            </ode>
+          </friction>
+        </surface>
       </collision>
+<<<<<<< HEAD
       <xacro:cylinder_inertia
         m="1.0"
@@ -128,33 +196,51 @@
         h="${wheel_width}"
         rpy="${pi/2} 0 0"/>
+=======
+      <inertial>
+        <mass value="1.0"/>
+        <inertia
+          ixx="0.002" ixy="0" ixz="0"
+          iyy="0.002" iyz="0"
+          izz="0.004"/>
+      </inertial>
+>>>>>>> b2d86b1 (Fixing URDF)
     </link>
-    <joint name="${prefix}_joint" type="continuous">
-      <parent link="base_footprint"/>
-      <child link="${prefix}_link"/>
-      <!-- wheel center is wheel_radius above ground -->
-      <origin xyz="${x} ${y} ${wheel_radius}" rpy="0 0 0"/>
+    <joint name="${name}_joint" type="continuous">
+      <parent link="base_link"/>
+      <child link="${name}_link"/>
+      <origin xyz="0 ${y} 0"/>
       <axis xyz="0 1 0"/>
-      <dynamics damping="0.05" friction="0.0"/>
+      <dynamics damping="0.05"/>
     </joint>
   </xacro:macro>
-  <xacro:wheel prefix="drivewhl_l" x="${wheel_xoff}" y="${ track/2}" />
-  <xacro:wheel prefix="drivewhl_r" x="${wheel_xoff}" y="${-track/2}" />
-  <!-- ===================== Swivel caster ===================== -->
-  <link name="caster_swivel_link">
+  <xacro:drive_wheel name="drivewhl_l" y="${ track/2}"/>
+  <xacro:drive_wheel name="drivewhl_r" y="${-track/2}"/>
+  <!-- ===================================================== -->
+  <!-- Ball caster (4 cm sphere)                              -->
+  <!-- ===================================================== -->
+  <link name="ball_caster_link">
     <visual>
-      <origin xyz="0 0 0" rpy="0 0 0"/>
-      <geometry>
-        <cylinder radius="0.008" length="0.03"/>
+      <geometry>
+        <sphere radius="${ball_radius}"/>
       </geometry>
       <material name="wheel_grey"/>
     </visual>
     <collision>
-      <origin xyz="0 0 0" rpy="0 0 0"/>
-      <geometry>
-        <cylinder radius="0.008" length="0.03"/>
-      </geometry>
-    </collision>
-    <xacro:cylinder_inertia m="0.15" r="0.008" h="0.03"/>
-  </link>
+      <geometry>
+        <sphere radius="${ball_radius}"/>
+      </geometry>
+      <!-- NEW: low friction so it supports but doesn't brake/steer the robot -->
+      <surface>
+        <friction>
+          <ode>
+            <mu>0.2</mu>
+            <mu2>0.2</mu2>
+          </ode>
+        </friction>
+      </surface>
+    </collision>
+    <xacro:tiny_inertial m="0.5"/>
+  </link>
+<<<<<<< HEAD
   <joint name="caster_swivel_joint" type="continuous">
     <parent link="base_footprint"/>
@@ -198,88 +284,74 @@
   </link>
   <joint name="lidar_joint" type="fixed">
-    <parent link="base_link"/>
-    <child link="lidar_link"/>
-    <origin xyz="-0.112 0.0 0.565" rpy="0.0 0.0 0.0"/>
-  </joint>
-  <link name="eyecam_link">
-    <xacro:tiny_inertial m="0.05" i="1e-5"/>
-  </link>
+=======
+  <joint name="ball_caster_joint" type="fixed">
+    <parent link="base_link"/>
+    <child link="ball_caster_link"/>
+    <origin xyz="${ball_x} 0 ${ball_radius - wheel_radius}"/>
+  </joint>
+  <!-- ===================================================== -->
+  <!-- Sensors                                               -->
+  <!-- ===================================================== -->
+  <!-- started at 0.565 raised by 20 cm to clear body       -->
+  <link name="base_laser"><xacro:tiny_inertial m="0.05"/></link>
+  <joint name="base_laser_joint" type="fixed">
+>>>>>>> b2d86b1 (Fixing URDF)
+    <parent link="base_link"/>
+    <child link="base_laser"/>
+    <origin xyz="-0.112 0 0.53" rpy ="0 0 0"/>
+  </joint>
+  <gazebo reference="base_laser">
+    <sensor name="ld06_lidar" type="gpu_lidar">
+      <update_rate>10</update_rate>
+      <always_on>true</always_on>
+      <topic>/world/empty/model/k9_robot/ld06/scan</topic>
+      <pose>0 0 0 0 0 0</pose>
+      <visualize>true</visualize>
+      <lidar>
+        <scan>
+          <horizontal>
+            <samples>360</samples>
+            <min_angle>-3.14159</min_angle>
+            <max_angle>3.14159</max_angle>
+          </horizontal>
+        </scan>
+        <range>
+          <min>0.02</min>
+          <max>12.0</max>
+        </range>
+      </lidar>
+      <always_on>true</always_on>
+      <visualize>true</visualize>
+    </sensor>
+  </gazebo>
+  <link name="eyecam_link"><xacro:tiny_inertial m="0.05"/></link>
   <joint name="eyecam_joint" type="fixed">
     <parent link="base_link"/>
     <child link="eyecam_link"/>
-    <origin xyz="0.366 0.0 0.67" rpy="0.0 0.0 0.0"/>
-  </joint>
-  <link name="3dcam_link">
-    <xacro:tiny_inertial m="0.10" i="2e-5"/>
-  </link>
+    <origin xyz="0.366 0 0.67"/>
+  </joint>
+  <link name="3dcam_link"><xacro:tiny_inertial m="0.10"/></link>
   <joint name="3dcam_joint" type="fixed">
     <parent link="base_link"/>
     <child link="3dcam_link"/>
-    <origin xyz="0.206 0.0 0.255" rpy="0.0 0.0 0.0"/>
-  </joint>
-  <link name="l_ear_link">
-    <xacro:tiny_inertial m="0.02" i="5e-6"/>
-  </link>
-  <joint name="l_ear_joint" type="fixed">
-    <parent link="base_link"/>
-    <child link="l_ear_link"/>
-    <origin xyz="0.35 0.045 0.725" rpy="0.0 0.65 0.0"/>
-  </joint>
-  <link name="r_ear_link">
-    <xacro:tiny_inertial m="0.02" i="5e-6"/>
-  </link>
-  <joint name="r_ear_joint" type="fixed">
-    <parent link="base_link"/>
-    <child link="r_ear_link"/>
-    <origin xyz="0.35 -0.045 0.725" rpy="0.0 0.65 0.0"/>
-  </joint>
-  <!-- ===================== Gazebo Sim extensions ===================== -->
-  <!-- Wheel / caster contact: give the drive wheels explicit friction too -->
-  <gazebo reference="drivewhl_l_link">
-    <surface>
-      <friction>
-        <ode>
-          <mu>1.1</mu>
-          <mu2>0.9</mu2>
-        </ode>
-      </friction>
-    </surface>
-  </gazebo>
-  <gazebo reference="drivewhl_r_link">
-    <surface>
-      <friction>
-        <ode>
-          <mu>1.1</mu>
-          <mu2>0.9</mu2>
-        </ode>
-      </friction>
-    </surface>
-  </gazebo>
-  <gazebo reference="caster_wheel_link">
-    <surface>
-      <friction>
-        <ode>
-          <mu>0.3</mu>
-          <mu2>0.15</mu2>
-        </ode>
-      </friction>
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
Commit message: Update after bug fix

File: src/k9_robot/src/description/k9.urdf (robot description, URDF)
Before this commit: robot k9_robot, 10 links, 9 joints
Links:
- added link l_ear_link, mass 0.05; visual box size=0.015 0.02 0.03; visual cylinder length=2.0 radius=0.01
- added link r_ear_link, mass 0.05; visual box size=0.015 0.02 0.03; visual cylinder length=2.0 radius=0.01
Joints:
- added joint l_ear_joint: type revolute, parent base_link, child l_ear_link, origin xyz=0.165 0.04 0.74 rpy=0.0 0.25 0.0, axis 0 0 1, limit lower=-0.2 upper=0.6 effort=0.1 velocity=10
- added joint r_ear_joint: type revolute, parent base_link, child r_ear_link, origin xyz=0.165 -0.04 0.74 rpy=0.0 0.25 0.0, axis 0 0 1, limit lower=-0.6 upper=0.2 effort=0.1 velocity=10

File: src/k9_robot/src/description/k9.urdf.xacro (robot description, xacro)
@@ -203,5 +203,5 @@
       <update_rate>10</update_rate>
       <always_on>true</always_on>
-      <topic>/scan</topic>
+      <topic>/world/empty/model/k9_robot/ld06/scan</topic>
       <pose>0 0 0 0 0 0</pose>
       <visualize>true</visualize>
@@ -248,7 +248,7 @@
   </visual>
   <visual name="l_ear_beam_visual">
-    <origin xyz="1.0 0 0" rpy="0 0 0"/>
+    <origin xyz="1.0 0 0" rpy="0 ${pi/2} 0"/>
     <geometry>
-      <cone radius="0.01" length="2.0"/>
+      <cylinder radius="0.01" length="2.0"/>
     </geometry>
     <material name="k9_beam_material">
@@ -260,11 +260,5 @@
   </visual>
   <!-- Inertia -->
-  <xacro:box_inertia
-    m="0.05"
-    x="0.015"
-    y="0.02"
-    z="0.03"
-    o_xyz="0 0 0"
-    o_rpy="0 0 0"/>
+  <xacro:tiny_inertial m="0.05"/>
 </link>
 <joint name="l_ear_joint" type="revolute">
@@ -290,7 +284,7 @@
   </visual>
   <visual name="r_ear_beam_visual">
-    <origin xyz="1.0 0 0" rpy="0 0 0"/>
+    <origin xyz="1.0 0 0" rpy="0 ${pi/2} 0"/>
     <geometry>
-      <cone radius="0.01" length="2.0"/>
+      <cylinder radius="0.01" length="2.0"/>
     </geometry>
     <material name="k9_beam_material">
@@ -301,11 +295,5 @@
     <transparency>0.6</transparency>
   </visual>
-  <xacro:box_inertia
-    m="0.05"
-    x="0.015"
-    y="0.02"
-    z="0.03"
-    o_xyz="0 0 0"
-    o_rpy="0 0 0"/>
+  <xacro:tiny_inertial m="0.05"/>
 </link>
 <joint name="r_ear_joint" type="revolute">
