Commit message: Added IMU

File: src/k9_robot/src/description/k9.urdf (robot description, URDF)
Before this commit: robot k9_robot, 12 links, 11 joints
Links:
- added link imu_link, mass 0.02
Joints:
- added joint imu_link_joint: type fixed, parent base_link, child imu_link, origin xyz=0 0 0.16 rpy=0 0 0

File: src/k9_robot/src/description/k9.urdf.xacro (robot description, xacro)
@@ -1,4 +1,10 @@
 <?xml version="1.0"?>
 <robot name="k9_robot" xmlns:xacro="http://ros.org/wiki/xacro">
+  <!-- ===================================================== -->
+  <!-- To generate SDF for Gazebo Sim                        -->
+  <!-- ros2 run xacro xacro k9.urdf.xacro > k9.urdf          -->
+  <!-- gz sdf -p k9.urdf > k9_raw.sdf                        -->
+  <!-- python3 patch_friction.py k9_raw.sdf k9_robot.sdf     -->
+  <!-- ===================================================== -->
   <!-- ===================================================== -->
   <!-- Materials                                             -->
@@ -37,4 +43,96 @@
         izz="1e-4"/>
     </inertial>
+  </xacro:macro>
+  <!-- ===================================================== -->
+  <!-- IMU (Gazebo Sim) helper macro                          -->
+  <!-- ===================================================== -->
+  <xacro:macro name="k9_add_imu" params="
+    parent_link
+    imu_link:=imu_link
+    xyz:='0 0 0'
+    rpy:='0 0 0'
+    update_rate:=200
+    accel_noise:=0.02
+    gyro_noise:=0.002
+    accel_bias:=0.0
+    gyro_bias:=0.0
+  ">
+    <!-- A tiny link to carry the IMU sensor -->
+    <link name="${imu_link}">
+      <inertial>
+        <origin xyz="0 0 0" rpy="0 0 0"/>
+        <mass value="0.02"/>
+        <inertia ixx="1e-6" ixy="0" ixz="0" iyy="1e-6" iyz="0" izz="1e-6"/>
+      </inertial>
+    </link>
+    <joint name="${imu_link}_joint" type="fixed">
+      <parent link="${parent_link}"/>
+      <child link="${imu_link}"/>
+      <origin xyz="${xyz}" rpy="${rpy}"/>
+    </joint>
+    <!-- Gazebo Sim sensor definition -->
+    <gazebo reference="${imu_link}">
+      <sensor name="${imu_link}_sensor" type="imu">
+        <topic>/k9/imu</topic>
+        <always_on>true</always_on>
+        <visualize>false</visualize>
+        <update_rate>${update_rate}</update_rate>
+        <!-- Noise model (tune these to feel like your BNO080) -->
+        <imu>
+          <angular_velocity>
+            <x>
+              <noise type="gaussian">
+                <mean>0.0</mean>
+                <stddev>${gyro_noise}</stddev>
+                <bias_mean>${gyro_bias}</bias_mean>
+                <bias_stddev>0.0</bias_stddev>
+              </noise>
+            </x>
+            <y>
+              <noise type="gaussian">
+                <mean>0.0</mean>
+                <stddev>${gyro_noise}</stddev>
+                <bias_mean>${gyro_bias}</bias_mean>
+                <bias_stddev>0.0</bias_stddev>
+              </noise>
+            </y>
+            <z>
+              <noise type="gaussian">
+                <mean>0.0</mean>
+                <stddev>${gyro_noise}</stddev>
+                <bias_mean>${gyro_bias}</bias_mean>
+                <bias_stddev>0.0</bias_stddev>
+              </noise>
+            </z>
+          </angular_velocity>
+          <linear_acceleration>
+            <x>
+              <noise type="gaussian">
+                <mean>0.0</mean>
+                <stddev>${accel_noise}</stddev>
+                <bias_mean>${accel_bias}</bias_mean>
+                <bias_stddev>0.0</bias_stddev>
+              </noise>
+            </x>
+            <y>
+              <noise type="gaussian">
+                <mean>0.0</mean>
+                <stddev>${accel_noise}</stddev>
+                <bias_mean>${accel_bias}</bias_mean>
+                <bias_stddev>0.0</bias_stddev>
+              </noise>
+            </y>
+            <z>
+              <noise type="gaussian">
+                <mean>0.0</mean>
+                <stddev>${accel_noise}</stddev>
+                <bias_mean>${accel_bias}</bias_mean>
+                <bias_stddev>0.0</bias_stddev>
+              </noise>
+            </z>
+          </linear_acceleration>
+        </imu>
+      </sensor>
+    </gazebo>
   </xacro:macro>
   <!-- ===================================================== -->
@@ -305,4 +403,11 @@
   <dynamics friction="0.1" damping="0.1"/>
 </joint>
+<xacro:k9_add_imu parent_link="base_link"
+                  imu_link="imu_link"
+                  xyz="0 0 0.16"
+                  rpy="0 0 0"
+                  update_rate="200"
+                  accel_noise="0.01"
+                  gyro_noise="0.001"/>
   <!-- ===================================================== -->
   <!-- Gazebo Diff Drive (gz-sim, Jazzy)                     -->

Commit message: Added camera

File: src/k9_robot/src/description/k9.urdf (robot description, URDF)
Before this commit: robot k9_robot, 13 links, 12 joints
Links:
- added link oakd_link, mass 0.05
- link l_ear_link: geometry visual box size=0.015 0.02 0.03
- link r_ear_link: geometry visual box size=0.015 0.02 0.03
Joints:
- added joint oakd_link_joint: type fixed, parent base_link, child oakd_link, origin xyz=0.206 0 0.255 rpy=0 0 0

File: src/k9_robot/src/description/k9.urdf.xacro (robot description, xacro)
@@ -137,4 +137,59 @@
   </xacro:macro>
   <!-- ===================================================== -->
+  <!-- OAK-D Lite-ish RGBD -> PointCloud (Gazebo Sim)         -->
+  <!-- ===================================================== -->
+  <xacro:macro name="k9_add_oakd_pointcloud" params="
+    parent_link
+    oak_link:=oakd_link
+    xyz:='0 0 0'
+    rpy:='0 0 0'
+    width:=640
+    height:=400
+    update_rate:=30
+    hfov:=1.3962634
+    near:=0.20
+    far:=8.0
+    depth_noise_stddev:=0.01
+    gz_topic:='/oak'
+    frame_id:='oak_depth_frame'">
+    <!-- A tiny link to carry the camera sensor -->
+    <link name="${oak_link}">
+      <inertial>
+        <origin xyz="0 0 0" rpy="0 0 0"/>
+        <mass value="0.05"/>
+        <inertia ixx="1e-5" ixy="0" ixz="0" iyy="1e-5" iyz="0" izz="1e-5"/>
+      </inertial>
+    </link>
+    <joint name="${oak_link}_joint" type="fixed">
+      <parent link="${parent_link}"/>
+      <child link="${oak_link}"/>
+      <origin xyz="${xyz}" rpy="${rpy}"/>
+    </joint>
+    <gazebo reference="${oak_link}">
+      <sensor name="${oak_link}_rgbd" type="rgbd_camera">
+        <always_on>true</always_on>
+        <visualize>false</visualize>
+        <update_rate>${update_rate}</update_rate>
+        <topic>${gz_topic}</topic>
+        <camera>
+          <horizontal_fov>${hfov}</horizontal_fov>
+          <image>
+            <width>${width}</width>
+            <height>${height}</height>
+          </image>
+          <clip>
+            <near>${near}</near>
+            <far>${far}</far>
+          </clip>
+          <noise>
+            <type>gaussian</type>
+            <mean>0.0</mean>
+            <stddev>0.003</stddev>
+          </noise>
+        </camera>
+      </sensor>
+    </gazebo>
+  </xacro:macro>
+  <!-- ===================================================== -->
   <!-- Frames                                                -->
   <!-- ===================================================== -->
@@ -322,133 +377,113 @@
   </joint>
   <!-- ******************** LEFT EAR ****************************** -->
-<link name="l_ear_link">
-  <!-- Visual (for Gazebo visualisation) -->
-  <visual name="l_ear_visual">
-    <origin xyz="0 0 0" rpy="0 0 0"/>
-    <geometry>
-      <box size="0.015 0.02 0.03"/>
-    </geometry>
-    <material name="k9_ear_emissive">
-      <ambient>0 0 0 1</ambient>
-      <diffuse>0 0 0 1</diffuse>
-      <emissive>0 0 0 1</emissive> <!-- will be driven by Gazebo -->
-    </material>
-  </visual>
-  <visual name="l_ear_beam_visual">
-    <origin xyz="1.0075 0 0" rpy="0 ${pi/2} 0"/>
-    <geometry>
-      <cylinder radius="0.01" length="2.0"/>
-    </geometry>
-    <material name="k9_beam_material">
-      <ambient>0 0 0 1</ambient>
-      <diffuse>0 0 0 1</diffuse>
-      <emissive>0 1 0 1</emissive>
-    </material>
-    <transparency>0.6</transparency>
-  </visual>
-  <!-- Inertia -->
-  <xacro:tiny_inertial m="0.05"/>
-</link>
-<gazebo reference="l_ear_link">
-  <sensor name="l_ear_tof" type="ray">
-    <pose>0.0075 0 0 0 0 0</pose>
-    <update_rate>30</update_rate>
-    <always_on>true</always_on>
-    <visualize>true</visualize>
-    <topic>/l_ear/scan</topic>
-    <ray>
-      <scan>
-        <horizontal>
-          <samples>1</samples>
-          <resolution>1</resolution>
-          <min_angle>0</min_angle>
-          <max_angle>0</max_angle>
-        </horizontal>
-      </scan>
-      <range>
-        <min>0.02</min>
-        <max>2.0</max>
-        <resolution>0.001</resolution>
-      </range>
-    </ray>
-  </sensor>
-</gazebo>
-<joint name="l_ear_joint" type="revolute">
-  <parent link="base_link"/>
-  <child link="l_ear_link"/>
-  <origin xyz="0.165 0.04 0.74" rpy="0.0 0.25 0.0"/>
-  <axis xyz="0 0 1"/>
-  <limit lower="-0.2" upper="0.6" effort="0.1" velocity="10"/>
-  <dynamics friction="0.1" damping="0.1"/>
-</joint>
-<!-- ******************** RIGHT EAR ****************************** -->
-<link name="r_ear_link">
-  <visual name="r_ear_visual">
-    <origin xyz="0 0 0" rpy="0 0 0"/>
-    <geometry>
-      <box size="0.015 0.02 0.03"/>
-    </geometry>
-    <material name="k9_ear_emissive">
-      <ambient>0 0 0 1</ambient>
-      <diffuse>0 0 0 1</diffuse>
-      <emissive>0 0 0 1</emissive>
-    </material>
-  </visual>
-  <visual name="r_ear_beam_visual">
-    <origin xyz="1.0075 0 0" rpy="0 ${pi/2} 0"/>
-    <geometry>
-      <cylinder radius="0.01" length="2.0"/>
-    </geometry>
-    <material name="k9_beam_material">
-      <ambient>0 0 0 1</ambient>
-      <diffuse>0 0 0 1</diffuse>
-      <emissive>0 1 0 1</emissive>
-    </material>
-    <transparency>0.6</transparency>
-  </visual>
-  <xacro:tiny_inertial m="0.05"/>
-</link>
-<gazebo reference="r_ear_link">
-  <sensor name="r_ear_tof" type="ray">
-    <pose>0.0075 0 0 0 0 0</pose>
-    <update_rate>30</update_rate>
-    <always_on>true</always_on>
-    <visualize>true</visualize>
-    <topic>/r_ear/scan</topic>
-    <ray>
-      <scan>
-        <horizontal>
-          <samples>1</samples>
-          <resolution>1</resolution>
-          <min_angle>0</min_angle>
-          <max_angle>0</max_angle>
-        </horizontal>
-      </scan>
-      <range>
-        <min>0.02</min>
-        <max>2.0</max>
-        <resolution>0.001</resolution>
-      </range>
-    </ray>
-  </sensor>
-</gazebo>
-<joint name="r_ear_joint" type="revolute">
-  <parent link="base_link"/>
-  <child link="r_ear_link"/>
-  <origin xyz="0.165 -0.04 0.74" rpy="0.0 0.25 0.0"/>
-  <axis xyz="0 0 1"/>
-  <limit lower="-0.6" upper="0.2" effort="0.1" velocity="10"/>
-  <dynamics friction="0.1" damping="0.1"/>
-</joint>
-<<<<<<< Updated upstream
-<xacro:k9_add_imu parent_link="base_link"
-                  imu_link="imu_link"
-                  xyz="0 0 0.16"
-                  rpy="0 0 0"
-                  update_rate="200"
-                  accel_noise="0.01"
-                  gyro_noise="0.001"/>
-=======
->>>>>>> Stashed changes
+  <link name="l_ear_link">
+    <!-- Visual (for Gazebo visualisation) -->
+    <visual name="l_ear_visual">
+      <origin xyz="0 0 0" rpy="0 0 0"/>
+      <geometry>
+        <box size="0.015 0.02 0.03"/>
+      </geometry>
+      <material name="k9_ear_emissive">
+        <ambient>0 0 0 1</ambient>
+        <diffuse>0 0 0 1</diffuse>
+        <emissive>0 0 0 1</emissive> <!-- will be driven by Gazebo -->
+      </material>
+    </visual>
+    <xacro:tiny_inertial m="0.05"/>
+  </link>
+  <gazebo reference="l_ear_link">
+    <sensor name="l_ear_tof" type="gpu_lidar">
+      <pose>0.0075 0 0 0 0 0</pose>
+      <update_rate>30</update_rate>
+      <always_on>true</always_on>
+      <visualize>true</visualize>
+      <topic>/l_ear/scan</topic>
+      <lidar>
+        <scan>
+          <horizontal>
+            <samples>1</samples>
+            <resolution>1</resolution>
+            <min_angle>0</min_angle>
+            <max_angle>0</max_angle>
+          </horizontal>
+        </scan>
+        <range>
+          <min>0.02</min>
+          <max>2.0</max>
+          <resolution>0.001</resolution>
+        </range>
+      </lidar>
+    </sensor>
+  </gazebo>
+  <joint name="l_ear_joint" type="revolute">
+    <parent link="base_link"/>
+    <child link="l_ear_link"/>
+    <origin xyz="0.165 0.04 0.74" rpy="0.0 0.25 0.0"/>
+    <axis xyz="0 0 1"/>
+    <limit lower="-0.2" upper="0.6" effort="0.1" velocity="10"/>
+    <dynamics friction="0.1" damping="0.1"/>
+  </joint>
+  <!-- ******************** RIGHT EAR ****************************** -->
+  <link name="r_ear_link">
+    <visual name="r_ear_visual">
+      <origin xyz="0 0 0" rpy="0 0 0"/>
+      <geometry>
+        <box size="0.015 0.02 0.03"/>
+      </geometry>
+      <material name="k9_ear_emissive">
+        <ambient>0 0 0 1</ambient>
+        <diffuse>0 0 0 1</diffuse>
+        <emissive>0 0 0 1</emissive>
+      </material>
+    </visual>
+    <xacro:tiny_inertial m="0.05"/>
+  </link>
+  <gazebo reference="r_ear_link">
+    <sensor name="r_ear_tof" type="gpu_lidar">
+      <pose>0.0075 0 0 0 0 0</pose>
+      <update_rate>30</update_rate>
+      <always_on>true</always_on>
+      <visualize>true</visualize>
+      <topic>/r_ear/scan</topic>
+      <lidar>
+        <scan>
+          <horizontal>
+            <samples>1</samples>
+            <resolution>1</resolution>
+            <min_angle>0</min_angle>
+            <max_angle>0</max_angle>
+          </horizontal>
+        </scan>
+        <range>
+          <min>0.02</min>
+          <max>2.0</max>
+          <resolution>0.001</resolution>
+        </range>
+      </lidar>
+    </sensor>
+  </gazebo>
+  <joint name="r_ear_joint" type="revolute">
+    <parent link="base_link"/>
+    <child link="r_ear_link"/>
+    <origin xyz="0.165 -0.04 0.74" rpy="0.0 0.25 0.0"/>
+    <axis xyz="0 0 1"/>
+    <limit lower="-0.6" upper="0.2" effort="0.1" velocity="10"/>
+    <dynamics friction="0.1" damping="0.1"/>
+  </joint>
+  <xacro:k9_add_imu
+    parent_link="base_link"
+    imu_link="imu_link"
+    xyz="0 0 0.16"
+    rpy="0 0 0"
+    update_rate="200"
+    accel_noise="0.01"
+    gyro_noise="0.001"/>
+  <xacro:k9_add_oakd_pointcloud
+    parent_link="base_link"
+    oak_link="oakd_link"
+    xyz="0.206 0 0.255"
+    rpy="0 0 0"
+    gz_topic="/oak"
+    frame_id="oak_depth_frame"/>
   <!-- ===================================================== -->
   <!-- Gazebo Diff Drive (gz-sim, Jazzy)                     -->

Commit message: Refine camera position

File: src/k9_robot/src/description/k9.urdf (robot description, URDF)
Before this commit: robot k9_robot, 14 links, 13 joints
Joints:
- joint oakd_link_joint: origin xyz=0.206 0 0.255 rpy=0 0 0 -> xyz=0.26 0 0.255 rpy=0 0 0

File: src/k9_robot/src/description/k9.urdf.xacro (robot description, xacro)
@@ -482,5 +482,5 @@
     parent_link="base_link"
     oak_link="oakd_link"
-    xyz="0.206 0 0.255"
+    xyz="0.26 0 0.255"
     rpy="0 0 0"
     gz_topic="/oak"

Commit message: Fixing ears

File: src/k9_robot/src/description/k9.urdf (robot description, URDF)
Before this commit: robot k9_robot, 14 links, 13 joints
Joints:
- joint l_ear_joint: limit lower=-0.2 upper=0.6 effort=0.1 velocity=10 -> lower=-0.2 upper=0.6 effort=2.0 velocity=10; origin xyz=0.165 0.04 0.74 rpy=0.0 0.25 0.0 -> xyz=0.27 0.0425 0.67 rpy=0.0 0.25 0.0
- joint r_ear_joint: limit lower=-0.6 upper=0.2 effort=0.1 velocity=10 -> lower=-0.6 upper=0.2 effort=2.0 velocity=10; origin xyz=0.165 -0.04 0.74 rpy=0.0 0.25 0.0 -> xyz=0.27 -0.0425 0.67 rpy=0.0 0.25 0.0

File: src/k9_robot/src/description/k9.urdf.xacro (robot description, xacro)
@@ -152,5 +152,5 @@
     depth_noise_stddev:=0.01
     gz_topic:='/oak'
-    frame_id:='oak_depth_frame'">
+    frame_id:='oakd_link'">
     <!-- A tiny link to carry the camera sensor -->
     <link name="${oak_link}">
@@ -419,8 +419,8 @@
     <parent link="base_link"/>
     <child link="l_ear_link"/>
-    <origin xyz="0.165 0.04 0.74" rpy="0.0 0.25 0.0"/>
+    <origin xyz="0.27 0.0425 0.67" rpy="0.0 0.25 0.0"/>
     <axis xyz="0 0 1"/>
-    <limit lower="-0.2" upper="0.6" effort="0.1" velocity="10"/>
-    <dynamics friction="0.1" damping="0.1"/>
+    <limit lower="-0.2" upper="0.6" effort="2.0" velocity="10"/>
+    <dynamics friction="0.01" damping="0.01"/>
   </joint>
   <!-- ******************** RIGHT EAR ****************************** -->
@@ -466,8 +466,8 @@
     <parent link="base_link"/>
     <child link="r_ear_link"/>
-    <origin xyz="0.165 -0.04 0.74" rpy="0.0 0.25 0.0"/>
+    <origin xyz="0.27 -0.0425 0.67" rpy="0.0 0.25 0.0"/>
     <axis xyz="0 0 1"/>
-    <limit lower="-0.6" upper="0.2" effort="0.1" velocity="10"/>
-    <dynamics friction="0.1" damping="0.1"/>
+    <limit lower="-0.6" upper="0.2" effort="2.0" velocity="10"/>
+    <dynamics friction="0.01" damping="0.01"/>
   </joint>
   <!-- ===================================================== -->

Commit message: oakd frame fix

File: src/k9_robot/src/description/k9.urdf (robot description, URDF)
Before this commit: robot k9_robot, 14 links, 13 joints
Links:
- added link camera_depth_frame
Joints:
- added joint camera_depth_frame_joint: type fixed, parent oakd_link, child camera_depth_frame, origin xyz=0 0 0 rpy=0 0 0

File: src/k9_robot/src/description/k9.urdf.xacro (robot description, xacro)
@@ -166,4 +166,11 @@
       <origin xyz="${xyz}" rpy="${rpy}"/>
     </joint>
+    <!-- Depth frame used by Gazebo / depthimage_to_laserscan -->
+    <link name="camera_depth_frame"/>
+    <joint name="camera_depth_frame_joint" type="fixed">
+      <parent link="oakd_link"/>   <!-- or oakd_link / 3dcam_link, whichever is your camera body -->
+      <child  link="camera_depth_frame"/>
+      <origin xyz="0 0 0" rpy="0 0 0"/>
+    </joint>
     <gazebo reference="${oak_link}">
       <sensor name="${oak_link}_rgbd" type="rgbd_camera">

Commit message: Revised ear frames

File: src/k9_robot/src/description/k9.urdf (robot description, URDF)
Before this commit: robot k9_robot, 15 links, 14 joints
Joints:
- joint camera_depth_frame_joint: origin xyz=0 0 0 rpy=0 0 0 -> xyz=0 0 0 rpy=-1.5707963267948966 0 -1.5707963267948966

File: src/k9_robot/src/description/k9.urdf.xacro (robot description, xacro)
@@ -356,4 +356,6 @@
       <pose>0 0 0 0 0 0</pose>
       <visualize>true</visualize>
+      <gz_frame_id>base_laser</gz_frame_id>
+      <frame_id>base_laser</frame_id>
       <lidar>
         <scan>
@@ -406,4 +408,6 @@
       <visualize>true</visualize>
       <topic>/l_ear/scan</topic>
+      <gz_frame_id>l_ear_link</gz_frame_id>
+      <frame_id>l_ear_link</frame_id>
       <lidar>
         <scan>
@@ -453,4 +457,6 @@
       <visualize>true</visualize>
       <topic>/r_ear/scan</topic>
+      <gz_frame_id>r_ear_link</gz_frame_id>
+      <frame_id>r_ear_link</frame_id>
       <lidar>
         <scan>
